Commit message: Resolve mesh paths through package:// like ROS does
The robot loaded with all 22 joints and no geometry at all. urdf-loader
prepends the URDF's own directory to any filename that is not a
package:// URI, so the rewritten absolute paths became
/robots/ur5e/meshes/... and every mesh 404'd silently.

The URDF now keeps its package:// URIs exactly as ROS writes them, and
public/robots/robot_description/ mirrors that package. Any future robot's
URDF resolves on its own with no path rewriting, which is the point of
reading descriptions instead of adapting them.

The viewer also reports joints and meshes on screen. That readout is what
made the failure legible: '22 joints, 0 meshes' says immediately that the
chain is fine and the geometry is not.

File: edurobotics_frontend/frontend-react/public/robots/ur5e/ur5e_robotiq.urdf (robot description, URDF)
Before this commit: robot ur5e_robotiq2f85, 23 links, 22 joints
Links:
- link base_link_inertia: geometry visual mesh filename=package://robot_description/meshes/arms/ur5e/visual/base.glb
- link forearm_link: geometry visual mesh filename=package://robot_description/meshes/arms/ur5e/visual/forearm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
- link robotiq_85_base_link: geometry visual mesh filename=package://robot_description/meshes/grippers/robotiq/visual/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
- link robotiq_85_left_finger_link: geometry visual mesh filename=package://robot_description/meshes/grippers/robotiq/visual/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
- link robotiq_85_left_finger_tip_link: geometry visual mesh filename=package://robot_description/meshes/grippers/robotiq/visual/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
- link robotiq_85_left_inner_knuckle_link: geometry visual mesh filename=package://robot_description/meshes/grippers/robotiq/visual/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
- link robotiq_85_left_knuckle_link: geometry visual mesh filename=package://robot_description/meshes/grippers/robotiq/visual/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
- link robotiq_85_right_finger_link: geometry visual mesh filename=package://robot_description/meshes/grippers/robotiq/visual/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
- link robotiq_85_right_finger_tip_link: geometry visual mesh filename=package://robot_description/meshes/grippers/robotiq/visual/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
- link robotiq_85_right_inner_knuckle_link: geometry visual mesh filename=package://robot_description/meshes/grippers/robotiq/visual/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
- link robotiq_85_right_knuckle_link: geometry visual mesh filename=package://robot_description/meshes/grippers/robotiq/visual/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
- link robotiq_coupling_link: geometry visual mesh filename=package://robot_description/meshes/grippers/robotiq/visual/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
- link shoulder_link: geometry visual mesh filename=package://robot_description/meshes/arms/ur5e/visual/shoulde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
- link upper_arm_link: geometry visual mesh filename=package://robot_description/meshes/arms/ur5e/visual/upperar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
- link wrist_1_link: geometry visual mesh filename=package://robot_description/meshes/arms/ur5e/visual/wrist1.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
- link wrist_2_link: geometry visual mesh filename=package://robot_description/meshes/arms/ur5e/visual/wrist2.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
- link wrist_3_link: geometry visual mesh filename=package://robot_description/meshes/arms/ur5e/visual/wrist3.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
